File: pcb/FeederController/FeederController.kicad_sch (KiCad schematic)
At the start: 10 parts, among them U1 ESP32-Module

Commit message: Update PCB as below
* Adjusted placement of mounting holes to line up with LumenPnP staging plate.
* Added 2k4 P/U for SDA/SCL.
* GND plane stitching
Parts:
- added R1, R2: 2k4, Resistor_SMD:R_0603_1608Metric_Pad0.98x0.95mm_HandSolder, symbol Device:R_Small_US
Connections:
- net +3V3: now also R1.1, R2.1
- net SCL: now also R2.2
- net SDA: now also R1.2
Other:
- note added: "I2C pull-ups"

Commit message: Added a few DNP footprints for connecting two PCBs together using a single ESP32
Parts:
- added J35: EXT-I2C, Connector_PinHeader_2.54mm:PinHeader_1x04_P2.54mm_Vertical, symbol Connector:Conn_01x04_Male
Connections:
- net +3V3: now also J35.1 (Pin_1)
- net GND: now also J35.4 (Pin_4)
- net SCL: now also J35.2 (Pin_2)
- net SDA: now also J35.3 (Pin_3)
Changed lines of the file:
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@@
+    (stroke (width 0) (type default) (color 0 0 0 0))
+  )
+  (wire (pts (xy 78.74 144.78) (xy 85.09 144.78))
     (stroke (width 0) (type default) (color 0 0 0 0))
   )
@@
     (stroke (width 0) (type default) (color 0 0 0 0))
   )
+  (wire (pts (xy 78.74 152.4) (xy 80.01 152.4))
+    (stroke (width 0) (type default) (color 0 0 0 0))
+  )
   (wire (pts (xy 60.96 124.46) (xy 62.23 124.46))
     (stroke (width 0) (type default) (color 0 0 0 0))
@@
     (effects (font (size 1.27 1.27)) (justify right bottom))
   )
+  (label "SCL" (at 78.74 147.32 0)
+    (effects (font (size 1.27 1.27)) (justify left bottom))
+  )
   (label "SCL" (at 177.8 124.46 180)
     (effects (font (size 1.27 1.27)) (justify right bottom))
@@
     (effects (font (size 1.27 1.27)) (justify left bottom))
   )
+  (label "SDA" (at 78.74 149.86 0)
+    (effects (font (size 1.27 1.27)) (justify left bottom))
+  )
   (label "SCL" (at 213.36 124.46 180)
     (effects (font (size 1.27 1.27)) (justify right bottom))
@@
       (effects (font (size 1.27 1.27)) hide)
     )
+  )
+  (symbol (lib_id "Connector:Conn_01x04_Male") (at 73.66 147.32 0) (unit 1)
+    (in_bom yes) (on_board yes)
+    (property "Reference" "J35" (id 0) (at 77.47 138.43 0))
+    (property "Value" "EXT-I2C" (id 1) (at 77.47 140.97 0))
+    (property "Footprint" "Connector_PinHeader_2.54mm:PinHeader_1x04_P2.54mm_Vertical" (id 2) (at 73.66 147.32 0)
+      (effects (font (size 1.27 1.27)) hide)
+    )
+    (property "Datasheet" "~" (id 3) (at 73.66 147.32 0)
+      (effects (font (size 1.27 1.27)) hide)
+    )
+    (pin "1")
+    (pin "2")
+    (pin "3")
+    (pin "4")
   )
   (symbol (lib_id "power:+3V3") (at 128.27 88.9 0) (unit 1)
@@
     (pin "2")
   )
+  (symbol (lib_id "power:GND") (at 80.01 152.4 0) (unit 1)
+    (in_bom yes) (on_board yes)
+    (property "Reference" "#PWR0103" (id 0) (at 80.01 158.75 0)
+      (effects (font (size 1.27 1.27)) hide)
+    )
+    (property "Value" "GND" (id 1) (at 77.47 156.21 0)
+      (effects (font (size 1.27 1.27)) (justify left))
+    )
+    (property "Footprint" "" (id 2) (at 80.01 152.4 0)
+      (effects (font (size 1.27 1.27)) hide)
+    )
+    (property "Datasheet" "" (id 3) (at 80.01 152.4 0)
+      (effects (font (size 1.27 1.27)) hide)
+    )
+    (pin "1")
+  )
   (symbol (lib_id "Mechanical:MountingHole") (at 58.42 189.23 0) (unit 1)
     (in_bom yes) (on_board yes) (fields_autoplaced)
@@
       (effects (font (size 1.27 1.27)) hide)
     )
+  )
+  (symbol (lib_id "power:+3V3") (at 85.09 144.78 0) (unit 1)
+    (in_bom yes) (on_board yes) (fields_autoplaced)
+    (property "Reference" "#PWR0104" (id 0) (at 85.09 148.59 0)
+      (effects (font (size 1.27 1.27)) hide)
+    )
+    (property "Value" "+3V3" (id 1) (at 85.09 139.7 0))
+    (property "Footprint" "" (id 2) (at 85.09 144.78 0)
+      (effects (font (size 1.27 1.27)) hide)
+    )
+    (property "Datasheet" "" (id 3) (at 85.09 144.78 0)
+      (effects (font (size 1.27 1.27)) hide)
+    )
+    (pin "1")
   )
   (symbol (lib_id "power:+3V3") (at 58.42 114.3 0) (unit 1)
@@
       (reference "#PWR0102") (unit 1) (value "GND") (footprint "")
     )
+    (path "/6f027b68-f5c9-4fc8-9766-427861905873"
+      (reference "#PWR0103") (unit 1) (value "GND") (footprint "")
+    )
+    (path "/9fd287ef-7357-4481-8ae0-6852dcd12ee6"
+      (reference "#PWR0104") (unit 1) (value "+3V3") (footprint "")
+    )
     (path "/191ccb4b-b935-4a99-9ccd-c92f2265624b/051b8f6a-584b-4cc1-8f17-4048b0c1a0b4"
       (reference "C1") (unit 1) (value "100nF") (footprint "Capacitor_SMD:C_0603_1608Metric_Pad1.08x0.95mm_HandSolder")
@@
       (reference "J34") (unit 1) (value "Feeder 32") (footprint "Connector_PinHeader_2.54mm:PinHeader_1x04_P2.54mm_Vertical")
     )
+    (path "/09fe9726-a1ec-4a3a-867a-188d385210f1"
+      (reference "J35") (unit 1) (value "EXT-I2C") (footprint "Connector_PinHeader_2.54mm:PinHeader_1x04_P2.54mm_Vertical")
+    )
     (path "/83084769-073a-41bd-9515-0bb9974896f2/ea645089-0040-4db0-ad82-6187112e402c"
       (reference "L1") (unit 1) (value "0.47uH") (footprint "Inductor_SMD:L_0603_1608Metric_Pad1.05x0.95mm_HandSolder")
@@
       (reference "R14") (unit 1) (value "10K") (footprint "Resistor_SMD:R_0603_1608Metric_Pad0.98x0.95mm_HandSolder")
     )
+    (path "/191ccb4b-b935-4a99-9ccd-c92f2265624b/7bb8446b-730f-422e-8a1f-82f77f35ae66"
+      (reference "R15") (unit 1) (value "10K") (footprint "Resistor_SMD:R_0603_1608Metric_Pad0.98x0.95mm_HandSolder")
+    )
+    (path "/191ccb4b-b935-4a99-9ccd-c92f2265624b/c5353bab-6942-498e-a03b-2a8ebbadb837"
+      (reference "R16") (unit 1) (value "10K") (footprint "Resistor_SMD:R_0603_1608Metric_Pad0.98x0.95mm_HandSolder")
+    )
+    (path "/191ccb4b-b935-4a99-9ccd-c92f2265624b/30307dab-11a5-4fe7-999e-05a3c316ea79"
+      (reference "R17") (unit 1) (value "10K") (footprint "Resistor_SMD:R_0603_1608Metric_Pad0.98x0.95mm_HandSolder")
+    )
+    (path "/191ccb4b-b935-4a99-9ccd-c92f2265624b/9ef127f4-6604-4e51-9060-0a5ac547bde3"
+      (reference "R18") (unit 1) (value "10K") (footprint "Resistor_SMD:R_0603_1608Metric_Pad0.98x0.95mm_HandSolder")
+    )
+    (path "/a82e31d2-26ac-4cb7-8053-72f9fc91d5bf/c769a380-b7a5-4701-8f51-1684b116bafc"
+      (reference "R19") (unit 1) (value "10K") (footprint "Resistor_SMD:R_0603_1608Metric_Pad0.98x0.95mm_HandSolder")
+    )
+    (path "/a82e31d2-26ac-4cb7-8053-72f9fc91d5bf/9d571d20-99ec-429e-a321-8982be849846"
+      (reference "R20") (unit 1) (value "10K") (footprint "Resistor_SMD:R_0603_1608Metric_Pad0.98x0.95mm_HandSolder")
+    )
+    (path "/a82e31d2-26ac-4cb7-8053-72f9fc91d5bf/c9ad4651-e1c8-45af-9130-278b87544087"
+      (reference "R21") (unit 1) (value "10K") (footprint "Resistor_SMD:R_0603_1608Metric_Pad0.98x0.95mm_HandSolder")
+    )
     (path "/191ccb4b-b935-4a99-9ccd-c92f2265624b/99cc2aae-550c-4f21-8a43-557a2da7105c"
       (reference "RN1") (unit 1) (value "220R") (footprint "Resistor_SMD:R_Array_Concave_4x0402")
@@
     )
     (path "/191ccb4b-b935-4a99-9ccd-c92f2265624b/a24eefd9-fb06-4d6a-86b7-85dbf7843557"
-      (reference "U3") (unit 1) (value "MCP23017") (footprint "Package_DFN_QFN:QFN-28-1EP_6x6mm_P0.65mm_EP4.25x4.25mm_ThermalVias")
+      (reference "U3") (unit 1) (value "MCP23017") (footprint "Package_DFN_QFN:QFN-28-1EP_6x6mm_P0.65mm_EP4.25x4.25mm")
     )
     (path "/83084769-073a-41bd-9515-0bb9974896f2/9f7650b8-b650-416b-8f29-e353db57ba37"
@@
     )
     (path "/a82e31d2-26ac-4cb7-8053-72f9fc91d5bf/6173f17e-e10a-420a-905e-60271ee066f7"
-      (reference "U7") (unit 1) (value "MCP23017_ML") (footprint "Package_DFN_QFN:QFN-28-1EP_6x6mm_P0.65mm_EP4.25x4.25mm_ThermalVias")
-    )
-  )
+      (reference "U7") (unit 1) (value "MCP23017_ML") (footprint "Package_DFN_QFN:QFN-28-1EP_6x6mm_P0.65mm_EP4.25x4.25mm")
+    )
+  )
