File: pcb/FeederController/servo2.kicad_sch (KiCad schematic)
At the start: 32 parts, among them J19 Feeder 17, J20 Feeder 18, J21 Feeder 19, J22 Feeder 20, J23 Feeder 21, J24 Feeder 22, J25 Feeder 23, J26 Feeder 24, J27 Feeder 25, J28 Feeder 26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

Commit message: Update PCB as below
* Adjusted placement of mounting holes to line up with LumenPnP staging plate.
* Added 2k4 P/U for SDA/SCL.
* GND plane stitching
Parts:
- renumbered R8 to R10, R9 to R11, R10 to R12, R11 to R13, R12 to R14, R7 to R9

Commit message: Added a few DNP footprints for connecting two PCBs together using a single ESP32
Parts:
- added R19, R20, R21: 10K, Resistor_SMD:R_0603_1608Metric_Pad0.98x0.95mm_HandSolder, symbol Device:R_Small_US
- U7: footprint Package_DFN_QFN:QFN-28-1EP_6x6mm_P0.65mm_EP4.25x4.25mm_ThermalVias -> Package_DFN_QFN:QFN-28-1EP_6x6mm_P0.65mm_EP4.25x4.25mm
Connections:
- net +3V3: now also R19.1, R20.1, R21.1
- net at U7.12 (A1): now also R21.2
- net at U6.2 (A1): now also R19.2
- net at U6.3 (A2): now also R20.2
- no-connect marks 7 -> 4
Other:
- note added: "DNP"
Changed lines of the file:
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@@
 (kicad_sch (version 20211123) (generator eeschema)
   (paper "A4")
+  (junction (at 13.97 168.91) (diameter 0) (color 0 0 0 0)
+  )
   (junction (at 45.72 34.29) (diameter 0) (color 0 0 0 0)
   )
+  (junction (at 15.24 67.31) (diameter 0) (color 0 0 0 0)
+  )
+  (junction (at 15.24 64.77) (diameter 0) (color 0 0 0 0)
+  )
   (junction (at 45.72 29.21) (diameter 0) (color 0 0 0 0)
   )
@@
   (junction (at 13.97 146.05) (diameter 0) (color 0 0 0 0)
   )
-  (no_connect (at 27.94 168.91))
   (no_connect (at 27.94 77.47))
   (no_connect (at 27.94 72.39))
-  (no_connect (at 27.94 67.31))
   (no_connect (at 27.94 74.93))
-  (no_connect (at 27.94 69.85))
   (no_connect (at 27.94 166.37))
   (wire (pts (xy 45.72 180.34) (xy 44.45 180.34))
@@
     (stroke (width 0) (type default) (color 0 0 0 0))
   )
-  (wire (pts (xy 13.97 153.67) (xy 13.97 171.45))
+  (wire (pts (xy 13.97 153.67) (xy 13.97 168.91))
     (stroke (width 0) (type default) (color 0 0 0 0))
   )
@@
     (stroke (width 0) (type default) (color 0 0 0 0))
   )
+  (wire (pts (xy 13.97 168.91) (xy 22.86 168.91))
+    (stroke (width 0) (type default) (color 0 0 0 0))
+  )
   (wire (pts (xy 73.66 69.85) (xy 73.66 73.66))
     (stroke (width 0) (type default) (color 0 0 0 0))
   )
+  (wire (pts (xy 15.24 67.31) (xy 15.24 64.77))
+    (stroke (width 0) (type default) (color 0 0 0 0))
+  )
   (wire (pts (xy 45.72 29.21) (xy 45.72 34.29))
     (stroke (width 0) (type default) (color 0 0 0 0))
@@
     (stroke (width 0) (type default) (color 0 0 0 0))
   )
+  (wire (pts (xy 15.24 67.31) (xy 15.24 69.85))
+    (stroke (width 0) (type default) (color 0 0 0 0))
+  )
+  (wire (pts (xy 22.86 67.31) (xy 15.24 67.31))
+    (stroke (width 0) (type default) (color 0 0 0 0))
+  )
   (wire (pts (xy 76.2 68.58) (xy 76.2 64.77))
     (stroke (width 0) (type default) (color 0 0 0 0))
@@
     (stroke (width 0) (type default) (color 0 0 0 0))
   )
+  (wire (pts (xy 13.97 168.91) (xy 13.97 171.45))
+    (stroke (width 0) (type default) (color 0 0 0 0))
+  )
   (wire (pts (xy 63.5 41.91) (xy 66.04 41.91))
     (stroke (width 0) (type default) (color 0 0 0 0))
@@
     (stroke (width 0) (type default) (color 0 0 0 0))
   )
+  (wire (pts (xy 15.24 69.85) (xy 22.86 69.85))
+    (stroke (width 0) (type default) (color 0 0 0 0))
+  )
   (wire (pts (xy 63.5 77.47) (xy 69.85 77.47))
     (stroke (width 0) (type default) (color 0 0 0 0))
@@
     (stroke (width 0) (type default) (color 0 0 0 0))
   )
+  (text "DNP" (at 26.67 69.85 0)
+    (effects (font (size 1.27 1.27)) (justify left bottom))
+  )
   (text "MCP23017 0x21" (at 15.24 163.83 0)
     (effects (font (size 1.27 1.27)) (justify left bottom))
   )
-  (text "PCA9685 0x41" (at 16.51 62.23 0)
+  (text "DNP" (at 22.86 167.64 0)
+    (effects (font (size 1.27 1.27)) (justify left bottom))
+  )
+  (text "PCA9685 0x41" (at 16.51 59.69 0)
+    (effects (font (size 1.27 1.27)) (justify left bottom))
+  )
+  (text "DNP" (at 26.67 67.31 0)
     (effects (font (size 1.27 1.27)) (justify left bottom))
   )
@@
       (effects (font (size 1.27 1.27)) (justify left))
     )
-    (property "Footprint" "Package_DFN_QFN:QFN-28-1EP_6x6mm_P0.65mm_EP4.25x4.25mm_ThermalVias" (id 2) (at 50.8 176.53 0)
+    (property "Footprint" "Package_DFN_QFN:QFN-28-1EP_6x6mm_P0.65mm_EP4.25x4.25mm" (id 2) (at 50.8 176.53 0)
       (effects (font (size 1.27 1.27)) (justify left) hide)
     )
@@
     (pin "1")
   )
+  (symbol (lib_id "Device:R_Small_US") (at 25.4 69.85 90) (unit 1)
+    (in_bom yes) (on_board yes)
+    (property "Reference" "R20" (id 0) (at 17.78 68.58 90))
+    (property "Value" "10K" (id 1) (at 21.59 68.58 90))
+    (property "Footprint" "Resistor_SMD:R_0603_1608Metric_Pad0.98x0.95mm_HandSolder" (id 2) (at 25.4 69.85 0)
+      (effects (font (size 1.27 1.27)) hide)
+    )
+    (property "Datasheet" "~" (id 3) (at 25.4 69.85 0)
+      (effects (font (size 1.27 1.27)) hide)
+    )
+    (property "Mouser" "279-CRGCQ0603F10K" (id 4) (at 25.4 69.85 90)
+      (effects (font (size 1.27 1.27)) hide)
+    )
+    (property "LCSC" "C98220" (id 5) (at 25.4 69.85 90)
+      (effects (font (size 1.27 1.27)) hide)
+    )
+    (pin "1")
+    (pin "2")
+  )
   (symbol (lib_id "power:GND") (at 212.09 77.47 270) (unit 1)
     (in_bom yes) (on_board yes)
@@
       (effects (font (size 1.27 1.27)) hide)
     )
+    (pin "1")
+    (pin "2")
+  )
+  (symbol (lib_id "Device:R_Small_US") (at 25.4 67.31 90) (unit 1)
+    (in_bom yes) (on_board yes)
+    (property "Reference" "R19" (id 0) (at 17.78 66.04 90))
+    (property "Value" "10K" (id 1) (at 21.59 66.04 90))
+    (property "Footprint" "Resistor_SMD:R_0603_1608Metric_Pad0.98x0.95mm_HandSolder" (id 2) (at 25.4 67.31 0)
+      (effects (font (size 1.27 1.27)) hide)
+    )
+    (property "Datasheet" "~" (id 3) (at 25.4 67.31 0)
+      (effects (font (size 1.27 1.27)) hide)
+    )
+    (property "Mouser" "279-CRGCQ0603F10K" (id 4) (at 25.4 67.31 90)
+      (effects (font (size 1.27 1.27)) hide)
+    )
+    (property "LCSC" "C98220" (id 5) (at 25.4 67.31 90)
+      (effects (font (size 1.27 1.27)) hide)
+    )
+    (pin "1")
+    (pin "2")
+  )
+  (symbol (lib_id "Device:R_Small_US") (at 25.4 168.91 90) (unit 1)
+    (in_bom yes) (on_board yes)
+    (property "Reference" "R21" (id 0) (at 17.78 167.64 90))
+    (property "Value" "10K" (id 1) (at 21.59 167.64 90))
+    (property "Footprint" "Resistor_SMD:R_0603_1608Metric_Pad0.98x0.95mm_HandSolder" (id 2) (at 25.4 168.91 0)
+      (effects (font (size 1.27 1.27)) hide)
+    )
+    (property "Datasheet" "~" (id 3) (at 25.4 168.91 0)
+      (effects (font (size 1.27 1.27)) hide)
+    )
+    (property "Mouser" "279-CRGCQ0603F10K" (id 4) (at 25.4 168.91 90)
+      (effects (font (size 1.27 1.27)) hide)
+    )
+    (property "LCSC" "C98220" (id 5) (at 25.4 168.91 90)
+      (effects (font (size 1.27 1.27)) hide)
+    )
